File: DMH_Slew_PCB_1/Core_Circuit.kicad_sch (KiCad schematic)
At the start: 0 parts

Commit message: Core circuit design in progress
Parts:
- added C5: 100pF, Capacitor_THT:C_Disc_D3.0mm_W2.0mm_P2.50mm, symbol Device:C
- added C6: 1uF, Capacitor_THT:C_Disc_D4.3mm_W1.9mm_P5.00mm, symbol Device:C
- added Q1: BC548, Package_TO_SOT_THT:TO-92L_Inline_Wide, symbol Transistor_BJT:BC548
- added Q2: BC558, Package_TO_SOT_THT:TO-92_Inline, symbol Transistor_BJT:BC558
- added Q3: BC558, Package_TO_SOT_THT:TO-92L_Inline_Wide, symbol Transistor_BJT:BC558
- added Q4: BC548, Package_TO_SOT_THT:TO-92_Inline, symbol Transistor_BJT:BC548
- added R10, R11: 10k, Resistor_THT:R_Axial_DIN0207_L6.3mm_D2.5mm_P7.62mm_Horizontal, symbol Device:R_US
- added R12: 1M, Resistor_THT:R_Axial_DIN0207_L6.3mm_D2.5mm_P7.62mm_Horizontal, symbol Device:R_US
- added R13: 470k, Resistor_THT:R_Axial_DIN0207_L6.3mm_D2.5mm_P7.62mm_Horizontal, symbol Device:R_US
- added R14: 3k3, Resistor_THT:R_Axial_DIN0207_L6.3mm_D2.5mm_P7.62mm_Horizontal, symbol Device:R_US
- added R15, R16, R17: 1k, Resistor_THT:R_Axial_DIN0207_L6.3mm_D2.5mm_P7.62mm_Horizontal, symbol Device:R_US
- added R18, R19, R2, R5, R9: 100k, Resistor_THT:R_Axial_DIN0207_L6.3mm_D2.5mm_P7.62mm_Horizontal, symbol Device:R_US
- added R20, R21, R22, R23, R6: 56k, Resistor_THT:R_Axial_DIN0207_L6.3mm_D2.5mm_P7.62mm_Horizontal, symbol Device:R_US
- added R7, R8: 2k7, Resistor_THT:R_Axial_DIN0207_L6.3mm_D2.5mm_P7.62mm_Horizontal, symbol Device:R_US
- added SW1: SW_SPDT, symbol Switch:SW_SPDT
- added U3: TL074, Package_DIP:DIP-14_W7.62mm_Socket, symbol Amplifier_Operational:TL074
Connections:
- new net: C5.1, Q1.1 (C), Q3.1 (C), R13.2, U3.9 (-)
- new net: Q1.2 (B), R16.2, R18.1, R20.1, R21.1
- new net: Q1.3 (E), Q2.3 (E), Q3.3 (E), Q4.3 (E), R14.2
- new net: C6.2, R15.1, R8.1, U3.14
- new net: R7.2, R8.2, R9.1, SW1.3 (C)
- new net: R6.2, U3.5 (+)
- new net: Q2.2 (B), R17.1, R19.2, R22.1, R23.1
- new net: C6.1, Q2.1 (C), Q4.1 (C), U3.13 (-)
- new net: R10.1, R9.2, SW1.1 (A)
- new net: R12.2, R13.1, U3.1
- new net: R11.1, SW1.2 (B)
- new net: R11.2, R12.1, U3.2 (-)
- new net: C5.2, R14.1, U3.8
- new net: R2.2, R5.1, U3.6 (-)
- new net: R5.2, R7.1, U3.7
- new net -12V: R18.2, R19.1
- new net GND: Q3.2 (B), Q4.2 (B), R10.2, R16.1, R17.2, R6.1, U3.10 (+), U3.12 (+), U3.3 (+)
- new net Input A: R2.1
- new net Output A: R15.2
