File: DMH_Slew_PCB_1_v2/DMH_Slew_PCB_1_v2.kicad_pcb (KiCad board)
At the start: 2 copper layers, 48 x 175 mm, 0 parts

Commit message: PCB 1 component placement ongoing
Parts:
- added C1: 47uF, Capacitor_THT:CP_Radial_D5.0mm_P2.00mm, B.Cu at (58.5, 47.5)
- added C10: 100nF, Capacitor_THT:C_Disc_D4.3mm_W1.9mm_P5.00mm, B.Cu at (151.6, 76.4)
- added C11: 100nF, Capacitor_THT:C_Disc_D4.3mm_W1.9mm_P5.00mm, B.Cu at (151.6, 79.8)
- added C12: 1uF, Capacitor_THT:C_Disc_D4.3mm_W1.9mm_P5.00mm, B.Cu at (271.2, 183.5)
- added C13: 220nF, Capacitor_THT:C_Disc_D4.3mm_W1.9mm_P5.00mm, B.Cu at (271.2, 186.9)
- added C14: 22nF, Capacitor_THT:C_Disc_D4.3mm_W1.9mm_P5.00mm, B.Cu at (281.9, 106.4)
- added C15: 220nF, Capacitor_THT:C_Disc_D4.3mm_W1.9mm_P5.00mm, B.Cu at (281.9, 109.8)
- added C16: 100nF, Capacitor_THT:C_Disc_D4.3mm_W1.9mm_P5.00mm, B.Cu at (66.4, 102.7)
- added C17: 100nF, Capacitor_THT:C_Disc_D4.3mm_W1.9mm_P5.00mm, B.Cu at (151.6, 86.7)
- added C18: 100nF, Capacitor_THT:C_Disc_D4.3mm_W1.9mm_P5.00mm, B.Cu at (151.6, 90.2)
- added C19: 100nF, Capacitor_THT:C_Disc_D4.3mm_W1.9mm_P5.00mm, B.Cu at (151.6, 93.6)
- added C2: 47uF, Capacitor_THT:CP_Radial_D5.0mm_P2.00mm, B.Cu at (93.5, 47.5)
- added C20: 100nF, Capacitor_THT:C_Disc_D4.3mm_W1.9mm_P5.00mm, B.Cu at (151.6, 97.1)
- added C21: 10pF, Capacitor_THT:C_Disc_D3.0mm_W2.0mm_P2.50mm, B.Cu at (221.7, 92.3)
- added C22: 220nF, Capacitor_THT:C_Disc_D4.3mm_W1.9mm_P5.00mm, B.Cu at (221.7, 102.9)
- added C23: 22nF, Capacitor_THT:C_Disc_D4.3mm_W1.9mm_P5.00mm, B.Cu at (221.7, 106.4)
- added C24: 2.2nF, Capacitor_THT:C_Disc_D4.3mm_W1.9mm_P5.00mm, B.Cu at (221.7, 109.8)
- added C25: 10pF, Capacitor_THT:C_Disc_D3.0mm_W2.0mm_P2.50mm, B.Cu at (221.7, 95.9)
- added C26: 10pF, Capacitor_THT:C_Disc_D3.0mm_W2.0mm_P2.50mm, B.Cu at (221.7, 99.4)
- added C27: 1uF, Capacitor_THT:C_Disc_D4.3mm_W1.9mm_P5.00mm, B.Cu at (301.7, 183.5)
- added C28: 220nF, Capacitor_THT:C_Disc_D4.3mm_W1.9mm_P5.00mm, B.Cu at (301.7, 186.9)
- added C3: 100nF, Capacitor_THT:C_Disc_D4.3mm_W1.9mm_P5.00mm, B.Cu at (151.6, 66.0)
- added C4: 100nF, Capacitor_THT:C_Disc_D4.3mm_W1.9mm_P5.00mm, B.Cu at (151.6, 69.5)
- added C5: 100nF, Capacitor_THT:C_Disc_D4.3mm_W1.9mm_P5.00mm, B.Cu at (63.8, 68.1)
- added C6: 10pF, Capacitor_THT:C_Disc_D3.0mm_W2.0mm_P2.50mm, B.Cu at (281.9, 92.3)
- added C7: 10pF, Capacitor_THT:C_Disc_D3.0mm_W2.0mm_P2.50mm, B.Cu at (281.9, 95.9)
- added C8: 10pF, Capacitor_THT:C_Disc_D3.0mm_W2.0mm_P2.50mm, B.Cu at (281.9, 99.4)
- added C9: 2.2nF, Capacitor_THT:C_Disc_D4.3mm_W1.9mm_P5.00mm, B.Cu at (281.9, 102.9)
- added D1: 1N4148, Diode_THT:D_DO-35_SOD27_P7.62mm_Horizontal, B.Cu at (271.2, 176.4)
- added D2: 1N4148, Diode_THT:D_DO-35_SOD27_P7.62mm_Horizontal, B.Cu at (271.2, 180.0)
- added D3: SB140, Diode_THT:D_DO-41_SOD81_P10.16mm_Horizontal, B.Cu at (78.0, 55.5)
- added D4: SB140, Diode_THT:D_DO-41_SOD81_P10.16mm_Horizontal, B.Cu at (61.8, 55.5)
- added D7: 1N4148, Diode_THT:D_DO-35_SOD27_P7.62mm_Horizontal, B.Cu at (301.7, 176.4)
- added D8: 1N4148, Diode_THT:D_DO-35_SOD27_P7.62mm_Horizontal, B.Cu at (301.7, 180.0)
- added J0: Conn_01x01, Connector_PinHeader_2.54mm:PinHeader_1x01_P2.54mm_Vertical, B.Cu at (53.3, 157.5)
- added J1: TS_Jack_6.35mm_Sw, SynthStuff:CUI_MJ-63052A, F.Cu at (58.5, 192.2)
- added J10: TS_Jack_6.35mm_Sw, SynthStuff:CUI_MJ-63052A, F.Cu at (91.5, 175.8)
- added J100: IDC_02x08, SynthStuff:IDC-Header_2x08_P2.54mm_Vertical_Eurorack, B.Cu at (83.9, 48.8)
- added J2: TS_Jack_6.35mm_Sw, SynthStuff:CUI_MJ-63052A, F.Cu at (75.0, 192.2)
- added J200: IDC_02x05, SynthStuff:IDC-Header_2x05_P2.54mm_Vertical_BackBone, B.Cu at (57.4, 177.2)
- added J3: TS_Jack_6.35mm_Sw, SynthStuff:CUI_MJ-63052A, F.Cu at (91.5, 192.2)
- added J4: TS_Jack_6.35mm_Sw, SynthStuff:CUI_MJ-63052A, F.Cu at (75.0, 159.2)
- added J5: TS_Jack_6.35mm_Sw, SynthStuff:CUI_MJ-63052A, F.Cu at (91.5, 159.2)
- added J50: Conn_01x08_PinHeader, Connector_PinHeader_2.54mm:PinHeader_1x08_P2.54mm_Vertical, F.Cu at (52.8, 50.0)
- added J51: Conn_01x08_PinHeader, Connector_PinHeader_2.54mm:PinHeader_1x08_P2.54mm_Vertical, F.Cu at (97.2, 76.0)
- added J6: TS_Jack_6.35mm_Sw, SynthStuff:CUI_MJ-63052A, F.Cu at (58.5, 208.8)
- added J60: Conn_01x08_PinHeader, Connector_PinHeader_2.54mm:PinHeader_1x08_P2.54mm_Vertical, F.Cu at (52.8, 102.0)
- added J61: Conn_01x08_PinHeader, Connector_PinHeader_2.54mm:PinHeader_1x08_P2.54mm_Vertical, F.Cu at (97.2, 128.0)
- added J7: TS_Jack_6.35mm_Sw, SynthStuff:CUI_MJ-63052A, F.Cu at (75.0, 208.8)
- added J8: TS_Jack_6.35mm_Sw, SynthStuff:CUI_MJ-63052A, F.Cu at (91.5, 208.8)
- added J9: TS_Jack_6.35mm_Sw, SynthStuff:CUI_MJ-63052A, F.Cu at (75.0, 175.8)
- added Q1: BC548, Package_TO_SOT_THT:TO-92L_Inline_Wide, B.Cu at (282.0, 82.5)
- added Q10: BC558, Package_TO_SOT_THT:TO-92L_Inline_Wide, B.Cu at (221.0, 124.7)
- added Q11: BC548, Package_TO_SOT_THT:TO-92L_Inline_Wide, B.Cu at (301.8, 191.9)
- added Q12: BC548, Package_TO_SOT_THT:TO-92L_Inline_Wide, B.Cu at (293.1, 185.0)
- added Q2: BC548, Package_TO_SOT_THT:TO-92L_Inline_Wide, B.Cu at (281.2, 119.0)
- added Q3: BC558, Package_TO_SOT_THT:TO-92L_Inline_Wide, B.Cu at (282.0, 88.2)
- added Q4: BC558, Package_TO_SOT_THT:TO-92L_Inline_Wide, B.Cu at (281.2, 124.7)
- added Q5: BC548, Package_TO_SOT_THT:TO-92L_Inline_Wide, B.Cu at (271.3, 191.9)
- added Q6: BC548, Package_TO_SOT_THT:TO-92L_Inline_Wide, B.Cu at (262.7, 185.0)
- added Q7: BC548, Package_TO_SOT_THT:TO-92L_Inline_Wide, B.Cu at (221.8, 82.5)
- added Q8: BC548, Package_TO_SOT_THT:TO-92L_Inline_Wide, B.Cu at (221.0, 119.0)
- added Q9: BC558, Package_TO_SOT_THT:TO-92L_Inline_Wide, B.Cu at (221.8, 88.2)
- added R1: 1k, Resistor_THT:R_Axial_DIN0207_L6.3mm_D2.5mm_P7.62mm_Horizontal, B.Cu at (314.3, 81.3)
- added R10: 100k, Resistor_THT:R_Axial_DIN0207_L6.3mm_D2.5mm_P7.62mm_Horizontal, B.Cu at (314.3, 109.6)
- added R11: 56k, Resistor_THT:R_Axial_DIN0207_L6.3mm_D2.5mm_P7.62mm_Horizontal, B.Cu at (314.3, 113.7)
- added R12: 56k, Resistor_THT:R_Axial_DIN0207_L6.3mm_D2.5mm_P7.62mm_Horizontal, B.Cu at (303.5, 81.3)
- added R13: 100k, Resistor_THT:R_Axial_DIN0207_L6.3mm_D2.5mm_P7.62mm_Horizontal, B.Cu at (303.5, 85.3)
- added R14: 1k, Resistor_THT:R_Axial_DIN0207_L6.3mm_D2.5mm_P7.62mm_Horizontal, B.Cu at (303.5, 89.4)
- added R15: 220k, Resistor_THT:R_Axial_DIN0207_L6.3mm_D2.5mm_P7.62mm_Horizontal, B.Cu at (303.5, 93.4)
- added R16: 100k, Resistor_THT:R_Axial_DIN0207_L6.3mm_D2.5mm_P7.62mm_Horizontal, B.Cu at (303.5, 97.5)
- added R17: 10k, Resistor_THT:R_Axial_DIN0207_L6.3mm_D2.5mm_P7.62mm_Horizontal, B.Cu at (303.5, 101.5)
- added R18: 1k8, Resistor_THT:R_Axial_DIN0207_L6.3mm_D2.5mm_P7.62mm_Horizontal, B.Cu at (303.5, 105.6)
- added R19: 1k8, Resistor_THT:R_Axial_DIN0207_L6.3mm_D2.5mm_P7.62mm_Horizontal, B.Cu at (303.5, 109.6)
- added R2: 100k, Resistor_THT:R_Axial_DIN0207_L6.3mm_D2.5mm_P7.62mm_Horizontal, B.Cu at (314.3, 85.3)
- added R20: 1k8, Resistor_THT:R_Axial_DIN0207_L6.3mm_D2.5mm_P7.62mm_Horizontal, B.Cu at (303.5, 113.7)
- added R21: 1k8, Resistor_THT:R_Axial_DIN0207_L6.3mm_D2.5mm_P7.62mm_Horizontal, B.Cu at (292.7, 81.3)
- added R22: 100k, Resistor_THT:R_Axial_DIN0207_L6.3mm_D2.5mm_P7.62mm_Horizontal, B.Cu at (292.7, 85.3)
- added R23: 100k, Resistor_THT:R_Axial_DIN0207_L6.3mm_D2.5mm_P7.62mm_Horizontal, B.Cu at (292.7, 89.4)
- added R24: 220k, Resistor_THT:R_Axial_DIN0207_L6.3mm_D2.5mm_P7.62mm_Horizontal, B.Cu at (292.7, 93.4)
- added R25: 220k, Resistor_THT:R_Axial_DIN0207_L6.3mm_D2.5mm_P7.62mm_Horizontal, B.Cu at (292.7, 97.5)
- added R26: 1k, Resistor_THT:R_Axial_DIN0207_L6.3mm_D2.5mm_P7.62mm_Horizontal, B.Cu at (292.7, 101.5)
- added R27: 100R, Resistor_THT:R_Axial_DIN0207_L6.3mm_D2.5mm_P7.62mm_Horizontal, B.Cu at (282.0, 142.0)
- added R28: 10k, Resistor_THT:R_Axial_DIN0207_L6.3mm_D2.5mm_P7.62mm_Horizontal, B.Cu at (282.0, 146.1)
- added R29: 10k, Resistor_THT:R_Axial_DIN0207_L6.3mm_D2.5mm_P7.62mm_Horizontal, B.Cu at (282.0, 150.1)
- added R30: 10k, Resistor_THT:R_Axial_DIN0207_L6.3mm_D2.5mm_P7.62mm_Horizontal, B.Cu at (282.0, 154.2)
- added R31: 4M7, Resistor_THT:R_Axial_DIN0207_L6.3mm_D2.5mm_P7.62mm_Horizontal, B.Cu at (282.0, 158.2)
- added R32: 4M7, Resistor_THT:R_Axial_DIN0207_L6.3mm_D2.5mm_P7.62mm_Horizontal, B.Cu at (282.0, 162.2)
- added R33: 100k, Resistor_THT:R_Axial_DIN0207_L6.3mm_D2.5mm_P7.62mm_Horizontal, B.Cu at (282.0, 166.3)
- added R34: 100k, Resistor_THT:R_Axial_DIN0207_L6.3mm_D2.5mm_P7.62mm_Horizontal, B.Cu at (282.0, 170.3)
- added R35: 1k, Resistor_THT:R_Axial_DIN0207_L6.3mm_D2.5mm_P7.62mm_Horizontal, B.Cu at (282.0, 174.4)
- added R36: 1k, Resistor_THT:R_Axial_DIN0207_L6.3mm_D2.5mm_P7.62mm_Horizontal, B.Cu at (282.0, 178.4)
- added R37: 1k8, Resistor_THT:R_Axial_DIN0207_L6.3mm_D2.5mm_P7.62mm_Horizontal, B.Cu at (282.0, 182.5)
- added R38: 2k2, Resistor_THT:R_Axial_DIN0207_L6.3mm_D2.5mm_P7.62mm_Horizontal, B.Cu at (282.0, 186.6)
- added R39: 10k, Resistor_THT:R_Axial_DIN0207_L6.3mm_D2.5mm_P7.62mm_Horizontal, B.Cu at (282.0, 190.6)
- added R40: 10k, Resistor_THT:R_Axial_DIN0207_L6.3mm_D2.5mm_P7.62mm_Horizontal, B.Cu at (282.0, 194.7)
- added R45: 1k, Resistor_THT:R_Axial_DIN0207_L6.3mm_D2.5mm_P7.62mm_Horizontal, B.Cu at (58.6, 109.6)
- added R47: 100k, Resistor_THT:R_Axial_DIN0207_L6.3mm_D2.5mm_P7.62mm_Horizontal, B.Cu at (254.0, 81.3)
- added R48: 100k, Resistor_THT:R_Axial_DIN0207_L6.3mm_D2.5mm_P7.62mm_Horizontal, B.Cu at (254.0, 85.3)
- added R49: 1k, Resistor_THT:R_Axial_DIN0207_L6.3mm_D2.5mm_P7.62mm_Horizontal, B.Cu at (58.6, 62.6)
- added R5: 100k, Resistor_THT:R_Axial_DIN0207_L6.3mm_D2.5mm_P7.62mm_Horizontal, B.Cu at (314.3, 89.4)
- added R50: 100k, Resistor_THT:R_Axial_DIN0207_L6.3mm_D2.5mm_P7.62mm_Horizontal, B.Cu at (254.0, 89.4)
- added R51: 100k, Resistor_THT:R_Axial_DIN0207_L6.3mm_D2.5mm_P7.62mm_Horizontal, B.Cu at (254.0, 93.4)
- added R52: 1k, Resistor_THT:R_Axial_DIN0207_L6.3mm_D2.5mm_P7.62mm_Horizontal, B.Cu at (254.0, 97.5)
- added R53: 56k, Resistor_THT:R_Axial_DIN0207_L6.3mm_D2.5mm_P7.62mm_Horizontal, B.Cu at (254.0, 101.5)
- added R54: 100k, Resistor_THT:R_Axial_DIN0207_L6.3mm_D2.5mm_P7.62mm_Horizontal, B.Cu at (254.0, 105.6)
- added R57: 100k, Resistor_THT:R_Axial_DIN0207_L6.3mm_D2.5mm_P7.62mm_Horizontal, B.Cu at (254.0, 109.6)
- added R59: 100k, Resistor_THT:R_Axial_DIN0207_L6.3mm_D2.5mm_P7.62mm_Horizontal, B.Cu at (254.0, 113.7)
- added R6: 100k, Resistor_THT:R_Axial_DIN0207_L6.3mm_D2.5mm_P7.62mm_Horizontal, B.Cu at (314.3, 93.4)
- added R60: 56k, Resistor_THT:R_Axial_DIN0207_L6.3mm_D2.5mm_P7.62mm_Horizontal, B.Cu at (243.3, 81.3)
- added R63: 220k, Resistor_THT:R_Axial_DIN0207_L6.3mm_D2.5mm_P7.62mm_Horizontal, B.Cu at (243.3, 85.3)
- added R64: 100k, Resistor_THT:R_Axial_DIN0207_L6.3mm_D2.5mm_P7.62mm_Horizontal, B.Cu at (243.3, 89.4)
- added R65: 100k, Resistor_THT:R_Axial_DIN0207_L6.3mm_D2.5mm_P7.62mm_Horizontal, B.Cu at (243.3, 93.4)
- added R66: 220k, Resistor_THT:R_Axial_DIN0207_L6.3mm_D2.5mm_P7.62mm_Horizontal, B.Cu at (243.3, 97.5)
- added R67: 1k8, Resistor_THT:R_Axial_DIN0207_L6.3mm_D2.5mm_P7.62mm_Horizontal, B.Cu at (243.3, 101.5)
- added R68: 1k8, Resistor_THT:R_Axial_DIN0207_L6.3mm_D2.5mm_P7.62mm_Horizontal, B.Cu at (243.3, 105.6)
- added R69: 1k, Resistor_THT:R_Axial_DIN0207_L6.3mm_D2.5mm_P7.62mm_Horizontal, B.Cu at (243.3, 109.6)
- added R7: 100k, Resistor_THT:R_Axial_DIN0207_L6.3mm_D2.5mm_P7.62mm_Horizontal, B.Cu at (314.3, 97.5)
- added R70: 1k, Resistor_THT:R_Axial_DIN0207_L6.3mm_D2.5mm_P7.62mm_Horizontal, B.Cu at (243.3, 113.7)
- added R71: 100k, Resistor_THT:R_Axial_DIN0207_L6.3mm_D2.5mm_P7.62mm_Horizontal, B.Cu at (232.5, 81.3)
- added R72: 100k, Resistor_THT:R_Axial_DIN0207_L6.3mm_D2.5mm_P7.62mm_Horizontal, B.Cu at (232.5, 85.3)
- added R73: 220k, Resistor_THT:R_Axial_DIN0207_L6.3mm_D2.5mm_P7.62mm_Horizontal, B.Cu at (232.5, 89.4)
- added R74: 10k, Resistor_THT:R_Axial_DIN0207_L6.3mm_D2.5mm_P7.62mm_Horizontal, B.Cu at (232.5, 93.4)
- added R75: 1k8, Resistor_THT:R_Axial_DIN0207_L6.3mm_D2.5mm_P7.62mm_Horizontal, B.Cu at (232.5, 97.5)
- added R76: 1k8, Resistor_THT:R_Axial_DIN0207_L6.3mm_D2.5mm_P7.62mm_Horizontal, B.Cu at (232.5, 101.5)
- added R77: 10k, Resistor_THT:R_Axial_DIN0207_L6.3mm_D2.5mm_P7.62mm_Horizontal, B.Cu at (312.5, 142.0)
- added R78: 1k8, Resistor_THT:R_Axial_DIN0207_L6.3mm_D2.5mm_P7.62mm_Horizontal, B.Cu at (312.5, 146.1)
- added R79: 4M7, Resistor_THT:R_Axial_DIN0207_L6.3mm_D2.5mm_P7.62mm_Horizontal, B.Cu at (312.5, 150.1)
- added R8: 100k, Resistor_THT:R_Axial_DIN0207_L6.3mm_D2.5mm_P7.62mm_Horizontal, B.Cu at (314.3, 101.5)
- added R80: 1k, Resistor_THT:R_Axial_DIN0207_L6.3mm_D2.5mm_P7.62mm_Horizontal, B.Cu at (312.5, 154.2)
- added R81: 10k, Resistor_THT:R_Axial_DIN0207_L6.3mm_D2.5mm_P7.62mm_Horizontal, B.Cu at (312.5, 158.2)
- added R82: 100k, Resistor_THT:R_Axial_DIN0207_L6.3mm_D2.5mm_P7.62mm_Horizontal, B.Cu at (312.5, 162.2)
- added R83: 100R, Resistor_THT:R_Axial_DIN0207_L6.3mm_D2.5mm_P7.62mm_Horizontal, B.Cu at (312.5, 166.3)
- added R84: 10k, Resistor_THT:R_Axial_DIN0207_L6.3mm_D2.5mm_P7.62mm_Horizontal, B.Cu at (312.5, 170.3)
- added R85: 10k, Resistor_THT:R_Axial_DIN0207_L6.3mm_D2.5mm_P7.62mm_Horizontal, B.Cu at (312.5, 174.4)
- added R86: 1k, Resistor_THT:R_Axial_DIN0207_L6.3mm_D2.5mm_P7.62mm_Horizontal, B.Cu at (312.5, 178.4)
- added R87: 2k2, Resistor_THT:R_Axial_DIN0207_L6.3mm_D2.5mm_P7.62mm_Horizontal, B.Cu at (312.5, 182.5)
- added R88: 10k, Resistor_THT:R_Axial_DIN0207_L6.3mm_D2.5mm_P7.62mm_Horizontal, B.Cu at (312.5, 186.6)
- added R89: 4M7, Resistor_THT:R_Axial_DIN0207_L6.3mm_D2.5mm_P7.62mm_Horizontal, B.Cu at (312.5, 190.6)
- added R9: 100k, Resistor_THT:R_Axial_DIN0207_L6.3mm_D2.5mm_P7.62mm_Horizontal, B.Cu at (314.3, 105.6)
- added R90: 100k, Resistor_THT:R_Axial_DIN0207_L6.3mm_D2.5mm_P7.62mm_Horizontal, B.Cu at (312.5, 194.7)
- added U1: TL074, Package_DIP:DIP-14_W7.62mm_Socket, B.Cu at (304.6, 117.8)
- added U10: LM4040LP-10, Package_TO_SOT_THT:TO-92_Inline, B.Cu at (65.2, 61.6)
- added U11: LM4040LP-10, Package_TO_SOT_THT:TO-92_Inline, B.Cu at (65.2, 108.7)
- added U2: TL074, Package_DIP:DIP-14_W7.62mm_Socket, B.Cu at (292.9, 117.8)
- added U3: TL074, Package_DIP:DIP-14_W7.62mm_Socket, B.Cu at (244.4, 117.8)
- added U4: TL074, Package_DIP:DIP-14_W7.62mm_Socket, B.Cu at (232.7, 117.8)
Routing:
- added copper zone on B.Cu, net GND
- added copper zone on F.Cu, net GND

Commit message: Updated Log circuit
Parts:
- R11, R12, R53, R60: value 56k -> 100k
Connections:
- J50 pad 1: +12V -> GND
- J60 pad 1: +12V -> GND
Changed lines of the file:
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@@
 			(layers "*.Cu" "*.Mask")
 			(remove_unused_layers no)
-			(net 2 "+12V")
+			(net 1 "GND")
 			(pinfunction "Pin_1")
 			(pintype "passive")
@@
 			(layers "*.Cu" "*.Mask")
 			(remove_unused_layers no)
-			(net 2 "+12V")
+			(net 1 "GND")
 			(pinfunction "Pin_1")
 			(pintype "passive")
@@
 			)
 		)
-		(property "Value" "56k"
+		(property "Value" "100k"
 			(at 3.81 -2.37 0)
 			(layer "B.Fab")
@@
 			)
 		)
-		(property "Value" "56k"
+		(property "Value" "100k"
 			(at 3.81 -2.37 0)
 			(layer "B.Fab")
@@
 			)
 		)
-		(property "Value" "56k"
+		(property "Value" "100k"
 			(at 3.81 -2.37 0)
 			(layer "B.Fab")
@@
 			)
 		)
-		(property "Value" "56k"
+		(property "Value" "100k"
 			(at 3.81 -2.37 0)
 			(layer "B.Fab")

Commit message: synced PCB 1 and sch
Parts:
- moved U1 223.9 mm to (84.4, 77.5)
- moved U2 223.9 mm to (72.7, 77.5)
- moved U4 164.4 mm to (68.5, 126.4)
- moved U3 153.2 mm to (91.7, 130.6)
- moved Q5 141.9 mm to (129.3, 193.1)
- moved R21 141.9 mm to (150.8, 82.4)
- moved R22 141.9 mm to (150.8, 86.4)
- moved R23 141.9 mm to (150.8, 90.5)
- moved R24 141.9 mm to (150.8, 94.5)
- moved R25 141.9 mm to (150.8, 98.6)
- moved R26 141.9 mm to (150.8, 102.6)
- moved R77 141.9 mm to (170.5, 143.1)
- moved R78 141.9 mm to (170.5, 147.2)
- moved R79 141.9 mm to (170.5, 151.2)
- moved R80 141.9 mm to (170.5, 155.2)
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