File: DMH_Slew_PCB_1_v3/DMH_Slew_PCB_1_v3.kicad_sch (KiCad schematic)
At the start: 47 parts, among them J1 TS_Jack_6.35mm_Sw, J2 Conn_01x08_PinHeader, J2 TS_Jack_6.35mm_Sw, J3 TS_Jack_6.35mm_Sw, Q1 BC548, Q2 BC548, Q3 BC558, Q4 BC558, SW1 SW_DPDT_3way, SW2 SW_DPDT, SW3 SPDT_OnOffOn, U1 TL074, U2 TL074

Commit message: Schematic redesign for submodules ongoig
Parts:
- removed unit 2 of J1
- removed unit 2 of J2
- removed unit 5 of J2
- removed unit 6 of J2
- removed unit 7 of J2
Connections:
- net A_Rng_Sw_p3_C: now reaches SW3.3 (C)
- net A_Rng_Sw_p3_C: no longer C15.2
- net A_Diff_Amp_S: now reaches C6.2, R8.1, U2.1
- net A_Diff_Amp_S: no longer SW2.1 (A)
- net A_CV_In_Jack_M: now reaches J2.T
- net A_CV_In_Jack_M: no longer R1.2
- net A_LinLog_Sw_p2_S: now reaches R10.2, R9.2
- net A_LinLog_Sw_p2_S: no longer SW2.2 (B)
- net A_LinLog_Sw_p5_S: now reaches R11.2, R12.2
- net A_LinLog_Sw_p5_S: no longer SW2.5 (B)
- net A_Rng_Sw_p1_C: now reaches SW3.1 (A)
- net A_Rng_Sw_p1_C: no longer C14.2
- net A CV Buff renamed A_CV_Buff_S
- net A CV Dest Sw renamed A_CV_Buff_C
- net A Fall CV renamed A_Fall_CV_S
- net A Fall Pot renamed A_Fall_CV_C
- net A Rise CV renamed A_Rise_CV_S
- net A Rise Pot renamed A_Rise_CV_C
- net Bus CV renamed A_In_Jack_TN_M
- net Input renamed A_Input_Jack_S
- net A_Input_Jack_S: no longer J1.T
- net Out A TN renamed A_Out_Jack_TN_M
- net Output renamed A_Out_Jack_S
- net A_Out_Jack_S: no longer J3.T, SW3.2 (B)
- new net A_CV_In_Jack_S: R1.2
- new net A_Diff_Amp_C: SW2.1 (A)
- new net A_Input_Jack_M: J1.T
- new net A_LinLog_Sw_p2_C: SW2.2 (B)
- new net A_LinLog_Sw_p5_C: SW2.5 (B)
- new net A_Out_Jack_C: SW3.2 (B)
- new net A_Out_Jack_M: J3.T
- new net A_Rng_Sw_p1_S: C14.2
- new net A_Rng_Sw_p3_S: C15.2
Other:
- note removed: "PCB 2"
- moved on the sheet: C14, C15, C6, C7, C8, C9, J1, J2, J3, Q1, Q2, Q3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

Commit message: V3 sch redesign ongoing
Parts:
- removed C14: 22nF, Capacitor_THT:C_Disc_D4.3mm_W1.9mm_P5.00mm, symbol Device:C
- removed C15: 220nF, Capacitor_THT:C_Disc_D4.3mm_W1.9mm_P5.00mm, symbol Device:C
- removed C6, C7, C8: 10pF, Capacitor_THT:C_Disc_D3.0mm_W2.0mm_P2.50mm, symbol Device:C
- removed C9: 2.2nF, Capacitor_THT:C_Disc_D4.3mm_W1.9mm_P5.00mm, symbol Device:C
- removed J1, J2, J3: TS_Jack_6.35mm_Sw, SynthStuff:CUI_MJ-63052A, symbol SynthStuff:TS_Jack_6.35mm_Sw
- removed Q1, Q2: BC548, Package_TO_SOT_THT:TO-92L_Inline_Wide, symbol Transistor_BJT:BC548
- removed Q3, Q4: BC558, Package_TO_SOT_THT:TO-92L_Inline_Wide, symbol Transistor_BJT:BC558
- removed R1, R14, R26: 1k, Resistor_THT:R_Axial_DIN0207_L6.3mm_D2.5mm_P7.62mm_Horizontal, symbol Device:R_US
- removed R10, R11, R12, R13, R16, R2, R22, R23, R5, R6, R7, R8, R9: 100k, Resistor_THT:R_Axial_DIN0207_L6.3mm_D2.5mm_P7.62mm_Horizontal, symbol Device:R_US
- removed R15, R24, R25: 220k, Resistor_THT:R_Axial_DIN0207_L6.3mm_D2.5mm_P7.62mm_Horizontal, symbol Device:R_US
- removed R17: 10k, Resistor_THT:R_Axial_DIN0207_L6.3mm_D2.5mm_P7.62mm_Horizontal, symbol Device:R_US
- removed R18, R19, R20, R21: 1k8, Resistor_THT:R_Axial_DIN0207_L6.3mm_D2.5mm_P7.62mm_Horizontal, symbol Device:R_US
- removed R3, R4: 56k, Resistor_THT:R_Axial_DIN0207_L6.3mm_D2.5mm_P7.62mm_Horizontal, symbol Device:R_US
- removed RV1, RV2: 100k, SynthStuff:Potentiometer_Alpha_RD901F-40-00D_Single_Vertical, symbol Device:R_Potentiometer_US
- removed SW1: SW_DPDT_3way, SynthStuff:Toggle_Switch_2_Poles_TE, symbol SynthStuff:Switch_DPDT
- removed SW2: SW_DPDT, SynthStuff:Toggle_Switch_2_Poles_TE, symbol SynthStuff:Switch_DPDT
- removed SW3: SPDT_OnOffOn, SynthStuff:Toggle_Switch_TE, symbol SynthStuff:SW_SPDT_OnOffOn
- removed U1, U2: TL074, Package_DIP:DIP-14_W7.62mm_Socket, symbol Amplifier_Operational:TL074
Other:
- sheet Core Circuit A ports: added none; removed Bus CV, Input, Output
- sheet Core Circuit B ports: added none; removed Input, Output
- sheet Power ports: added none; removed Bus CV
- sheet State Gate Outputs A ports: added none; removed Input, Output
- sheet State Gate Outputs B ports: added none; removed Input, Output
- note removed: "22pF in bb"
- note removed: "2x SPST switches"
