File: DMH_Slew_PCB_1_v3/Core_Circuit_A.kicad_sch (KiCad schematic)
At the start: 60 parts, among them J1 TS_Jack_6.35mm_Sw, J11 Conn_02x03_Top_Bottom, J12 Conn_02x06_Top_Bottom, J13 Conn_02x03_Top_Bottom, J14 Conn_02x03_Top_Bottom, J15 Conn_02x06_Top_Bottom, J16 Conn_02x03_Top_Bottom, J17 Conn_01x08, J18 Conn_01x08, J19 Conn_01x08, J2 TS_Jack_6.35mm_Sw, J20 Conn_01x08, J3 TS_Jack_6.35mm_Sw, Q1 BC548, Q2 BC548, Q3 BC558, Q4 BC558, SW1 SW_DPDT_3way, SW2 SW_DPDT, SW3 SPDT_OnOffOn, U1 TL074, U2 TL074

Commit message: Cleaned up old breadboarding notes
Other:
- note removed: "2x SPST switches"
Changed lines of the file:
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@@
 		(comment 1 "PCB for 5 cm Kosmo format synthesizer module")
-	)
-	(text "2x SPST switches"
-		(exclude_from_sim no)
-		(at 141.478 100.076 0)
-		(effects
-			(font
-				(size 1.27 1.27)
-			)
-		)
 	)
 	(junction
