File: DMH_Slew_PCB_1_v3/Core_Circuit_B.kicad_sch (KiCad schematic)
At the start: 60 parts, among them J21 Conn_02x03_Top_Bottom, J22 Conn_02x06_Top_Bottom, J23 Conn_02x03_Top_Bottom, J24 Conn_02x03_Top_Bottom, J25 Conn_02x06_Top_Bottom, J26 Conn_02x03_Top_Bottom, J27 Conn_01x08, J28 Conn_01x08, J29 Conn_01x08, J30 Conn_01x08, J6 TS_Jack_6.35mm_Sw, J7 TS_Jack_6.35mm_Sw, J8 TS_Jack_6.35mm_Sw, Q10 BC558, Q7 BC548, Q8 BC548, Q9 BC558, SW4 SW_DPDT_3way, SW5 SW_DPDT, SW6 SPDT_OnOffOn, U3 TL074, U4 TL074

Commit message: Cleaned up old breadboarding notes
Other:
- note removed: "2x SPST switches"
Changed lines of the file:
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@@
 		(comment 1 "PCB for 5 cm Kosmo format synthesizer module")
-	)
-	(text "2x SPST switches"
-		(exclude_from_sim no)
-		(at 141.478 100.076 0)
-		(effects
-			(font
-				(size 1.27 1.27)
-			)
-		)
 	)
 	(junction
