File: DMH_Slew_PANEL_v2/DMH_Slew_PANEL_v2.kicad_pcb (KiCad board)
At the start: 2 copper layers, 50 x 200 mm, 28 parts

Commit message: Generated Gerbers
Other:
- board text added: "Mk1.0 - March 2026"
- board text removed: "Mk1.0 - Month Year"
